File: stduinof429.sch (KiCad schematic (older format))
At the start: 22 parts, among them P1 Power, P11 CONN_01X03, P12 USB_OTG, P2 Analog, P3 Digital, P4 Digital, P5 CONN_1, P6 CONN_1, P7 CONN_1, P8 CONN_1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

Commit message: Porting from Kicad 4 to Kicad 5
Parts:
- C1, C2: footprint Capacitors_Tantalum_SMD:TantalC_SizeA_EIA-3216_HandSoldering -> Capacitor_Tantalum_SMD:CP_EIA-3216-18_Kemet-A_Pad1.58x1.35mm_HandSolder; symbol CP1_Small -> Device1:CP1_Small
- C27, C3, C4: footprint Capacitors_SMD:C_1210_HandSoldering -> Capacitor_SMD:C_1210_3225Metric_Pad1.42x2.65mm_HandSolder; symbol C_Small -> Device1:C_Small
- D1: footprint LEDs:LED_1206 -> LED_SMD:LED_1206_3216Metric_Pad1.42x1.75mm_HandSolder; symbol LED -> stduinof429-rescue:LED
- P1, P4: footprint Socket_Strips:Socket_Strip_Straight_1x08 -> Connector_PinSocket_2.54mm:PinSocket_1x08_P2.54mm_Vertical; symbol CONN_8 -> stduinof429-rescue:CONN_8
- P11: footprint Pin_Headers:Pin_Header_Straight_1x03 -> Connector_PinHeader_2.54mm:PinHeader_1x03_P2.54mm_Vertical; symbol CONN_01X03 -> stduinof429-rescue:CONN_01X03
- P12: symbol USB_OTG -> stduinof429-rescue:USB_OTG
- P2: footprint Socket_Strips:Socket_Strip_Straight_1x06 -> Connector_PinSocket_2.54mm:PinSocket_1x06_P2.54mm_Vertical; symbol CONN_6 -> stduinof429-rescue:CONN_6
- P3: footprint Socket_Strips:Socket_Strip_Straight_1x10 -> Connector_PinSocket_2.54mm:PinSocket_1x10_P2.54mm_Vertical; symbol CONN_10 -> stduinof429-rescue:CONN_10
- P5, P6, P7, P8, P9: symbol CONN_1 -> stduinof429-rescue:CONN_1
- R1, R2: footprint Resistors_SMD:R_1210_HandSoldering -> Resistor_SMD:R_1210_3225Metric_Pad1.42x2.65mm_HandSolder; symbol R_Small -> Device1:R_Small
- SW1: symbol SW_PUSH -> stduinof429-rescue:SW_PUSH
- U1: footprint TO_SOT_Packages_SMD:SOT-223 -> Package_TO_SOT_SMD:SOT-223; symbol AZ1117-3.3 -> Regulator_Linear1:AZ1117-3.3
- W1: footprint Wire_Pads:SolderWirePad_single_0-8mmDrill -> TestPoint:TestPoint_Pad_D2.0mm; symbol TEST_1P -> stduinof429-rescue:TEST_1P
Connections:
- wire segments 93 -> 109

Commit message: Added without the packages/kicad folder needed. All stuff is now on kicad sources and RetroBitLab Library
Parts:
- C1, C2: symbol Device1:CP1_Small -> stduinof429-rescue:CP1_Small-Device1-stduinof429-rescue
- C27, C3, C4: symbol Device1:C_Small -> stduinof429-rescue:C_Small-Device1-stduinof429-rescue
- D1: symbol stduinof429-rescue:LED -> stduinof429-rescue:LED-stduinof429-rescue
- P1, P4: symbol stduinof429-rescue:CONN_8 -> stduinof429-rescue:CONN_8-stduinof429-rescue
- P11: symbol stduinof429-rescue:CONN_01X03 -> stduinof429-rescue:CONN_01X03-stduinof429-rescue
- P12: symbol stduinof429-rescue:USB_OTG -> stduinof429-rescue:USB_OTG-stduinof429-rescue
- P2: symbol stduinof429-rescue:CONN_6 -> stduinof429-rescue:CONN_6-stduinof429-rescue
- P3: symbol stduinof429-rescue:CONN_10 -> stduinof429-rescue:CONN_10-stduinof429-rescue
- P5, P6, P7, P8, P9: symbol stduinof429-rescue:CONN_1 -> stduinof429-rescue:CONN_1-stduinof429-rescue
- R1, R2: symbol Device1:R_Small -> stduinof429-rescue:R_Small-Device1-stduinof429-rescue
- SW1: symbol stduinof429-rescue:SW_PUSH -> stduinof429-rescue:SW_PUSH-stduinof429-rescue
- U1: symbol Regulator_Linear1:AZ1117-3.3 -> stduinof429-rescue:AZ1117-3.3-Regulator_Linear1-stduinof429-rescue
- W1: symbol stduinof429-rescue:TEST_1P -> stduinof429-rescue:TEST_1P-stduinof429-rescue
Changed lines of the file:
@@
 EESchema Schematic File Version 4
-LIBS:stduinof429-cache
-EELAYER 26 0
+EELAYER 30 0
 EELAYER END
 $Descr A4 11693 8268
@@
 Sheet 1 2
 Title "STM32Duino429"
-Date "lun. 30 mars 2015"
-Rev "1.0"
+Date "2021-03-22"
+Rev "1.1"
 Comp "RetroBit Lab"
 Comment1 "Arduino Shield Layout"
@@
 $EndDescr
 $Comp
-L stduinof429-rescue:CONN_8 P1
+L stduinof429-rescue:CONN_8-stduinof429-rescue P1
 U 1 1 5517C2C1
 P 9725 1875
@@
 $EndComp
 $Comp
-L stduinof429-rescue:CONN_6 P2
+L stduinof429-rescue:CONN_6-stduinof429-rescue P2
 U 1 1 5517C323
 P 9725 2675
@@
 $EndComp
 $Comp
-L stduinof429-rescue:CONN_8 P4
+L stduinof429-rescue:CONN_8-stduinof429-rescue P4
 U 1 1 5517C366
 P 10050 2575
@@
 $EndComp
 $Comp
-L stduinof429-rescue:CONN_10 P3
+L stduinof429-rescue:CONN_10-stduinof429-rescue P3
 U 1 1 5517C46C
 P 10050 1575
@@
 AREF
 $Comp
-L power1:GND #PWR01
+L stduinof429-rescue:GND-power1-stduinof429-rescue #PWR01
 U 1 1 5517CC27
 P 10475 3100
@@
 $EndComp
 $Comp
-L power1:GND #PWR02
+L stduinof429-rescue:GND-power1-stduinof429-rescue #PWR02
 U 1 1 5517CC7B
 P 9300 3100
@@
 $EndComp
 $Comp
-L power1:+3.3V #PWR03
+L stduinof429-rescue:+3.3V-power1-stduinof429-rescue #PWR03
 U 1 1 5517CCDA
 P 9175 1350
@@
 A5(SCL)
 $Comp
-L stduinof429-rescue:CONN_1 P5
+L stduinof429-rescue:CONN_1-stduinof429-rescue P5
 U 1 1 551BBC06
 P 10875 650
@@
 $EndComp
 $Comp
-L stduinof429-rescue:CONN_1 P6
+L stduinof429-rescue:CONN_1-stduinof429-rescue P6
 U 1 1 551BBD10
 P 10950 650
@@
 $EndComp
 $Comp
-L stduinof429-rescue:CONN_1 P7
+L stduinof429-rescue:CONN_1-stduinof429-rescue P7
 U 1 1 551BBD30
 P 11025 650
@@
 $EndComp
 $Comp
-L stduinof429-rescue:CONN_1 P8
+L stduinof429-rescue:CONN_1-stduinof429-rescue P8
 U 1 1 551BBD52
 P 11100 650
@@
 Shield for Arduino that uses\nthe same pin disposition\nlike "Uno" board Rev 3.
 $Comp
-L Regulator_Linear1:AZ1117-3.3 U1
+L stduinof429-rescue:AZ1117-3.3-Regulator_Linear1-stduinof429-rescue U1
 U 1 1 5DA23390
 P 2250 2025
@@
 $EndComp
 $Comp
-L Device1:C_Small C3
+L stduinof429-rescue:C_Small-Device1-stduinof429-rescue C3
 U 1 1 5DA23506
 P 3000 2300
@@
 $EndComp
 $Comp
-L Device1:CP1_Small C2
+L stduinof429-rescue:CP1_Small-Device1-stduinof429-rescue C2
 U 1 1 5DA23553
 P 2700 2300
@@
 $EndComp
 $Comp
-L Device1:CP1_Small C1
+L stduinof429-rescue:CP1_Small-Device1-stduinof429-rescue C1
 U 1 1 5DA2358A
 P 1775 2300
@@
 $EndComp
 $Comp
-L power1:GND #PWR04
+L stduinof429-rescue:GND-power1-stduinof429-rescue #PWR04
 U 1 1 5DA238C8
 P 3000 2950
@@
 $EndComp
 $Comp
-L stduinof429-rescue:TEST_1P W1
+L stduinof429-rescue:TEST_1P-stduinof429-rescue W1
 U 1 1 5DA2393F
 P 2875 2800
@@
 $EndComp
 $Comp
-L stduinof429-rescue:LED D1
+L stduinof429-rescue:LED-stduinof429-rescue D1
 U 1 1 5DA239FC
 P 3300 2725
@@
 $EndComp
 $Comp
-L power1:GND #PWR05
+L stduinof429-rescue:GND-power1-stduinof429-rescue #PWR05
 U 1 1 5DA23A43
 P 3300 2950
@@
 $EndComp
 $Comp
-L Device1:R_Small R1
+L stduinof429-rescue:R_Small-Device1-stduinof429-rescue R1
 U 1 1 5DA23AF5
 P 3300 2300
@@
 VCC_3V3
 $Comp
-L power1:PWR_FLAG #FLG06
+L stduinof429-rescue:PWR_FLAG-power1-stduinof429-rescue #FLG06
 U 1 1 5DA24062
 P 3475 1500
@@
 VCC5V
 $Comp
-L power1:GND #PWR07
+L stduinof429-rescue:GND-power1-stduinof429-rescue #PWR07
 U 1 1 5DA242C3
 P 3150 1550
@@
 $EndComp
 $Comp
-L power1:PWR_FLAG #FLG08
+L stduinof429-rescue:PWR_FLAG-power1-stduinof429-rescue #FLG08
 U 1 1 5DA242F5
 P 2975 1500
@@
 VCC_3V3
 $Comp
-L Device1:R_Small R2
+L stduinof429-rescue:R_Small-Device1-stduinof429-rescue R2
 U 1 1 5DA28353
 P 6300 1975
@@
 	6300 1750 6300 1875
 $Comp
-L power1:GND #PWR09
+L stduinof429-rescue:GND-power1-stduinof429-rescue #PWR09
 U 1 1 5DA28681
 P 6300 2850
@@
 $EndComp
 $Comp
-L stduinof429-rescue:SW_PUSH SW1
+L stduinof429-rescue:SW_PUSH-stduinof429-rescue SW1
 U 1 1 5DA286C5
 P 6025 2550
@@
 	6025 2850 6300 2850
 $Comp
-L Device1:C_Small C4
+L stduinof429-rescue:C_Small-Device1-stduinof429-rescue C4
 U 1 1 5DA2889B
 P 6300 2550
@@
 $EndSheet
 $Comp
-L stduinof429-rescue:CONN_1 P9
+L stduinof429-rescue:CONN_1-stduinof429-rescue P9
 U 1 1 5DA49690
 P 11175 650
@@
 D12
 $Comp
-L power1:+5V #PWR010
+L stduinof429-rescue:+5V-power1-stduinof429-rescue #PWR010
 U 1 1 5DA371CC
 P 1375 1475
@@
 $EndComp
 $Comp
-L power1:PWR_FLAG #FLG011
+L stduinof429-rescue:PWR_FLAG-power1-stduinof429-rescue #FLG011
 U 1 1 5DA37249
 P 1275 1400
@@
 	1275 1475 1375 1475
 $Comp
-L power1:+3.3V #PWR012
+L stduinof429-rescue:+3.3V-power1-stduinof429-rescue #PWR012
 U 1 1 5DA38573
 P 3500 1900
@@
 VCC5V
 $Comp
-L stduinof429-rescue:CONN_01X03 P11
+L stduinof429-rescue:CONN_01X03-stduinof429-rescue P11
 U 1 1 5DA3B776
 P 1225 2025
@@
 $EndComp
 $Comp
-L power1:+5V #PWR013
+L stduinof429-rescue:+5V-power1-stduinof429-rescue #PWR013
 U 1 1 5DA3B7E5
 P 1425 1925
@@
 	1425 2125 1425 2350
 $Comp
-L stduinof429-rescue:USB_OTG P12
+L stduinof429-rescue:USB_OTG-stduinof429-rescue P12
 U 1 1 5DA3BD90
 P 9875 4575
@@
 NoConn ~ 9975 4875
 $Comp
-L power1:GND #PWR014
+L stduinof429-rescue:GND-power1-stduinof429-rescue #PWR014
 U 1 1 5DA3BEC3
 P 10075 5025
@@
 	9675 4875 9675 5000
 $Comp
-L Device1:C_Small C27
+L stduinof429-rescue:C_Small-Device1-stduinof429-rescue C27
 U 1 1 5DA3C280
 P 9900 5000
@@
 USB POWER PLUG
 $Comp
-L power1:PWR_FLAG #FLG015
+L stduinof429-rescue:PWR_FLAG-power1-stduinof429-rescue #FLG015
 U 1 1 5DA3D4AB
 P 9425 5000

Commit message: Created for rescue :-(
Parts:
- C1, C2: symbol stduinof429-rescue:CP1_Small-Device1-stduinof429-rescue -> stduinof429-rescue:CP1_Small-Device1-stduinof429-rescue-stduinof429-rescue
- C27, C3, C4: symbol stduinof429-rescue:C_Small-Device1-stduinof429-rescue -> stduinof429-rescue:C_Small-Device1-stduinof429-rescue-stduinof429-rescue
- D1: symbol stduinof429-rescue:LED-stduinof429-rescue -> stduinof429-rescue:LED-stduinof429-rescue-stduinof429-rescue
- P1, P4: symbol stduinof429-rescue:CONN_8-stduinof429-rescue -> stduinof429-rescue:CONN_8-stduinof429-rescue-stduinof429-rescue
- P11: symbol stduinof429-rescue:CONN_01X03-stduinof429-rescue -> stduinof429-rescue:CONN_01X03-stduinof429-rescue-stduinof429-rescue
- P12: symbol stduinof429-rescue:USB_OTG-stduinof429-rescue -> stduinof429-rescue:USB_OTG-stduinof429-rescue-stduinof429-rescue
- P2: symbol stduinof429-rescue:CONN_6-stduinof429-rescue -> stduinof429-rescue:CONN_6-stduinof429-rescue-stduinof429-rescue
- P3: symbol stduinof429-rescue:CONN_10-stduinof429-rescue -> stduinof429-rescue:CONN_10-stduinof429-rescue-stduinof429-rescue
- P5, P6, P7, P8, P9: symbol stduinof429-rescue:CONN_1-stduinof429-rescue -> stduinof429-rescue:CONN_1-stduinof429-rescue-stduinof429-rescue
- R1, R2: symbol stduinof429-rescue:R_Small-Device1-stduinof429-rescue -> stduinof429-rescue:R_Small-Device1-stduinof429-rescue-stduinof429-rescue
- SW1: symbol stduinof429-rescue:SW_PUSH-stduinof429-rescue -> stduinof429-rescue:SW_PUSH-stduinof429-rescue-stduinof429-rescue
- U1: symbol stduinof429-rescue:AZ1117-3.3-Regulator_Linear1-stduinof429-rescue -> stduinof429-rescue:AZ1117-3.3-Regulator_Linear1-stduinof429-rescue-stduinof429-rescue
- W1: symbol stduinof429-rescue:TEST_1P-stduinof429-rescue -> stduinof429-rescue:TEST_1P-stduinof429-rescue-stduinof429-rescue
Changed lines of the file:
@@
 $EndDescr
 $Comp
-L stduinof429-rescue:CONN_8-stduinof429-rescue P1
+L stduinof429-rescue:CONN_8-stduinof429-rescue-stduinof429-rescue P1
 U 1 1 5517C2C1
 P 9725 1875
@@
 $EndComp
 $Comp
-L stduinof429-rescue:CONN_6-stduinof429-rescue P2
+L stduinof429-rescue:CONN_6-stduinof429-rescue-stduinof429-rescue P2
 U 1 1 5517C323
 P 9725 2675
@@
 $EndComp
 $Comp
-L stduinof429-rescue:CONN_8-stduinof429-rescue P4
+L stduinof429-rescue:CONN_8-stduinof429-rescue-stduinof429-rescue P4
 U 1 1 5517C366
 P 10050 2575
@@
 $EndComp
 $Comp
-L stduinof429-rescue:CONN_10-stduinof429-rescue P3
+L stduinof429-rescue:CONN_10-stduinof429-rescue-stduinof429-rescue P3
 U 1 1 5517C46C
 P 10050 1575
@@
 AREF
 $Comp
-L stduinof429-rescue:GND-power1-stduinof429-rescue #PWR01
+L stduinof429-rescue:GND-power1-stduinof429-rescue-stduinof429-rescue #PWR01
 U 1 1 5517CC27
 P 10475 3100
@@
 $EndComp
 $Comp
-L stduinof429-rescue:GND-power1-stduinof429-rescue #PWR02
+L stduinof429-rescue:GND-power1-stduinof429-rescue-stduinof429-rescue #PWR02
 U 1 1 5517CC7B
 P 9300 3100
@@
 $EndComp
 $Comp
-L stduinof429-rescue:+3.3V-power1-stduinof429-rescue #PWR03
+L stduinof429-rescue:+3.3V-power1-stduinof429-rescue-stduinof429-rescue #PWR03
 U 1 1 5517CCDA
 P 9175 1350
@@
 A5(SCL)
 $Comp
-L stduinof429-rescue:CONN_1-stduinof429-rescue P5
+L stduinof429-rescue:CONN_1-stduinof429-rescue-stduinof429-rescue P5
 U 1 1 551BBC06
 P 10875 650
@@
 $EndComp
 $Comp
-L stduinof429-rescue:CONN_1-stduinof429-rescue P6
+L stduinof429-rescue:CONN_1-stduinof429-rescue-stduinof429-rescue P6
 U 1 1 551BBD10
 P 10950 650
@@
 $EndComp
 $Comp
-L stduinof429-rescue:CONN_1-stduinof429-rescue P7
+L stduinof429-rescue:CONN_1-stduinof429-rescue-stduinof429-rescue P7
 U 1 1 551BBD30
 P 11025 650
@@
 $EndComp
 $Comp
-L stduinof429-rescue:CONN_1-stduinof429-rescue P8
+L stduinof429-rescue:CONN_1-stduinof429-rescue-stduinof429-rescue P8
 U 1 1 551BBD52
 P 11100 650
@@
 Shield for Arduino that uses\nthe same pin disposition\nlike "Uno" board Rev 3.
 $Comp
-L stduinof429-rescue:AZ1117-3.3-Regulator_Linear1-stduinof429-rescue U1
+L stduinof429-rescue:AZ1117-3.3-Regulator_Linear1-stduinof429-rescue-stduinof429-rescue U1
 U 1 1 5DA23390
 P 2250 2025
@@
 $EndComp
 $Comp
-L stduinof429-rescue:C_Small-Device1-stduinof429-rescue C3
+L stduinof429-rescue:C_Small-Device1-stduinof429-rescue-stduinof429-rescue C3
 U 1 1 5DA23506
 P 3000 2300
@@
 $EndComp
 $Comp
-L stduinof429-rescue:CP1_Small-Device1-stduinof429-rescue C2
+L stduinof429-rescue:CP1_Small-Device1-stduinof429-rescue-stduinof429-rescue C2
 U 1 1 5DA23553
 P 2700 2300
@@
 $EndComp
 $Comp
-L stduinof429-rescue:CP1_Small-Device1-stduinof429-rescue C1
+L stduinof429-rescue:CP1_Small-Device1-stduinof429-rescue-stduinof429-rescue C1
 U 1 1 5DA2358A
 P 1775 2300
@@
 $EndComp
 $Comp
-L stduinof429-rescue:GND-power1-stduinof429-rescue #PWR04
+L stduinof429-rescue:GND-power1-stduinof429-rescue-stduinof429-rescue #PWR04
 U 1 1 5DA238C8
 P 3000 2950
@@
 $EndComp
 $Comp
-L stduinof429-rescue:TEST_1P-stduinof429-rescue W1
+L stduinof429-rescue:TEST_1P-stduinof429-rescue-stduinof429-rescue W1
 U 1 1 5DA2393F
 P 2875 2800
@@
 $EndComp
 $Comp
-L stduinof429-rescue:LED-stduinof429-rescue D1
+L stduinof429-rescue:LED-stduinof429-rescue-stduinof429-rescue D1
 U 1 1 5DA239FC
 P 3300 2725
@@
 $EndComp
 $Comp
-L stduinof429-rescue:GND-power1-stduinof429-rescue #PWR05
+L stduinof429-rescue:GND-power1-stduinof429-rescue-stduinof429-rescue #PWR05
 U 1 1 5DA23A43
 P 3300 2950
@@
 $EndComp
 $Comp
-L stduinof429-rescue:R_Small-Device1-stduinof429-rescue R1
+L stduinof429-rescue:R_Small-Device1-stduinof429-rescue-stduinof429-rescue R1
 U 1 1 5DA23AF5
 P 3300 2300
@@
 VCC_3V3
 $Comp
-L stduinof429-rescue:PWR_FLAG-power1-stduinof429-rescue #FLG06
+L stduinof429-rescue:PWR_FLAG-power1-stduinof429-rescue-stduinof429-rescue #FLG06
 U 1 1 5DA24062
 P 3475 1500
@@
 VCC5V
 $Comp
-L stduinof429-rescue:GND-power1-stduinof429-rescue #PWR07
+L stduinof429-rescue:GND-power1-stduinof429-rescue-stduinof429-rescue #PWR07
 U 1 1 5DA242C3
 P 3150 1550
@@
 $EndComp
 $Comp
-L stduinof429-rescue:PWR_FLAG-power1-stduinof429-rescue #FLG08
+L stduinof429-rescue:PWR_FLAG-power1-stduinof429-rescue-stduinof429-rescue #FLG08
 U 1 1 5DA242F5
 P 2975 1500
@@
 VCC_3V3
 $Comp
-L stduinof429-rescue:R_Small-Device1-stduinof429-rescue R2
+L stduinof429-rescue:R_Small-Device1-stduinof429-rescue-stduinof429-rescue R2
 U 1 1 5DA28353
 P 6300 1975
@@
 	6300 1750 6300 1875
 $Comp
-L stduinof429-rescue:GND-power1-stduinof429-rescue #PWR09
+L stduinof429-rescue:GND-power1-stduinof429-rescue-stduinof429-rescue #PWR09
 U 1 1 5DA28681
 P 6300 2850
@@
 $EndComp
 $Comp
-L stduinof429-rescue:SW_PUSH-stduinof429-rescue SW1
+L stduinof429-rescue:SW_PUSH-stduinof429-rescue-stduinof429-rescue SW1
 U 1 1 5DA286C5
 P 6025 2550
@@
 	6025 2850 6300 2850
 $Comp
-L stduinof429-rescue:C_Small-Device1-stduinof429-rescue C4
+L stduinof429-rescue:C_Small-Device1-stduinof429-rescue-stduinof429-rescue C4
 U 1 1 5DA2889B
 P 6300 2550
@@
 $EndSheet
 $Comp
-L stduinof429-rescue:CONN_1-stduinof429-rescue P9
+L stduinof429-rescue:CONN_1-stduinof429-rescue-stduinof429-rescue P9
 U 1 1 5DA49690
 P 11175 650
@@
 D12
 $Comp
-L stduinof429-rescue:+5V-power1-stduinof429-rescue #PWR010
+L stduinof429-rescue:+5V-power1-stduinof429-rescue-stduinof429-rescue #PWR010
 U 1 1 5DA371CC
 P 1375 1475
@@
 $EndComp
 $Comp
-L stduinof429-rescue:PWR_FLAG-power1-stduinof429-rescue #FLG011
+L stduinof429-rescue:PWR_FLAG-power1-stduinof429-rescue-stduinof429-rescue #FLG011
 U 1 1 5DA37249
 P 1275 1400
@@
 	1275 1475 1375 1475
 $Comp
-L stduinof429-rescue:+3.3V-power1-stduinof429-rescue #PWR012
+L stduinof429-rescue:+3.3V-power1-stduinof429-rescue-stduinof429-rescue #PWR012
 U 1 1 5DA38573
 P 3500 1900
@@
 VCC5V
 $Comp
-L stduinof429-rescue:CONN_01X03-stduinof429-rescue P11
+L stduinof429-rescue:CONN_01X03-stduinof429-rescue-stduinof429-rescue P11
 U 1 1 5DA3B776
 P 1225 2025
@@
 $EndComp
 $Comp
-L stduinof429-rescue:+5V-power1-stduinof429-rescue #PWR013
+L stduinof429-rescue:+5V-power1-stduinof429-rescue-stduinof429-rescue #PWR013
 U 1 1 5DA3B7E5
 P 1425 1925
@@
 	1425 2125 1425 2350
 $Comp
-L stduinof429-rescue:USB_OTG-stduinof429-rescue P12
+L stduinof429-rescue:USB_OTG-stduinof429-rescue-stduinof429-rescue P12
 U 1 1 5DA3BD90
 P 9875 4575
@@
 NoConn ~ 9975 4875
 $Comp
-L stduinof429-rescue:GND-power1-stduinof429-rescue #PWR014
+L stduinof429-rescue:GND-power1-stduinof429-rescue-stduinof429-rescue #PWR014
 U 1 1 5DA3BEC3
 P 10075 5025
@@
 	9675 4875 9675 5000
 $Comp
-L stduinof429-rescue:C_Small-Device1-stduinof429-rescue C27
+L stduinof429-rescue:C_Small-Device1-stduinof429-rescue-stduinof429-rescue C27
 U 1 1 5DA3C280
 P 9900 5000
@@
 USB POWER PLUG
 $Comp
-L stduinof429-rescue:PWR_FLAG-power1-stduinof429-rescue #FLG015
+L stduinof429-rescue:PWR_FLAG-power1-stduinof429-rescue-stduinof429-rescue #FLG015
 U 1 1 5DA3D4AB
 P 9425 5000
